Commit message: update new mesh locations in urdf

File: urdf/pan_tilt_adapter.xacro (robot description, xacro)
@@ -8,10 +8,10 @@
 			<visual>
 				<geometry>
-			  		<mesh filename="package://h4r_pantilt_adapter/meshes/basepart.dae"  />
+			  		<mesh filename="package://h4r_pantilt_adapter/meshes/v1_combined/base.dae"  />
 				</geometry>
 			</visual>
 			<collision name="pantilt_foot_link_collision">
 				<geometry>
-					<mesh filename="package://h4r_pantilt_adapter/meshes/basepart.dae"  />
+					<mesh filename="package://h4r_pantilt_adapter/meshes/v1_combined/base.dae"  />
 				</geometry>
 			</collision>
@@ -36,10 +36,10 @@
 			<visual>
 				<geometry>
-			  		<mesh filename="package://h4r_pantilt_adapter/meshes/centerpart.dae"  />
+			  		<mesh filename="package://h4r_pantilt_adapter/meshes/v1_combined/center.dae"  />
 				</geometry>
 			</visual>
 			<collision name="pantilt_center_link_collision">
 				<geometry>
-					<mesh filename="package://h4r_pantilt_adapter/meshes/centerpart.dae"  />
+					<mesh filename="package://h4r_pantilt_adapter/meshes/v1_combined/center.dae"  />
 				</geometry>
 			</collision>
@@ -64,10 +64,10 @@
 			<visual>
 				<geometry>
-			  		<mesh filename="package://h4r_pantilt_adapter/meshes/toppart.dae"  />
+			  		<mesh filename="package://h4r_pantilt_adapter/meshes/v1_combined/multicamera_mount.dae"  />
 				</geometry>
 			</visual>
 			<collision name="pantilt_top_link_collision">
 				<geometry>
-					<mesh filename="package://h4r_pantilt_adapter/meshes/toppart.dae"  />
+					<mesh filename="package://h4r_pantilt_adapter/meshes/v1_combined/multicamera_mount.dae"  />
 				</geometry>
 			</collision>

Commit message: update thermapp mount center and base

File: urdf/pan_tilt_adapter.xacro (robot description, xacro)
@@ -29,5 +29,5 @@
       <axis xyz="0 0 1"/>
       <limit lower="0" upper="1" effort="9" velocity="1" />
-      <origin xyz="0 0 0.0028" rpy="0 0 0" />
+      <origin xyz="0 0 0.0027" rpy="0 0 0" />
       <parent link="pantilt_base_link"/>
       <child link="pantilt_center_link"/>
@@ -57,5 +57,5 @@
       <axis xyz="1 0 0"/>
       <limit lower="0" upper="1" effort="9" velocity="1" />
-      <origin xyz="-0.022267 0 0.045495" rpy="0 0 3.14" />
+      <origin xyz="0.0223 0 0.0455" rpy="0 0 0" />
       <parent link="pantilt_center_link"/>
       <child link="pantilt_top_link"/>
