Commit message: fix limits in xacro

File: h4r_pantilt_descriptions/defs/pan_tilt_adapter.xacro (robot description, xacro)
@@ -28,5 +28,5 @@
 	<joint name="pantilt_pan_joint" type="revolute">
       <axis xyz="0 0 1"/>
-      <limit lower="0" upper="1" effort="9" velocity="1" />
+      <limit lower="0" upper="3.14" effort="9" velocity="1" />
       <origin xyz="0 0 0.0027" rpy="0 0 0" />
       <parent link="pantilt_base_link"/>
@@ -39,9 +39,9 @@
 				</geometry>
 			</visual>
-			<collision name="pantilt_center_link_collision">
+<!--			<collision name="pantilt_center_link_collision">
 				<geometry>
 					<mesh filename="package://h4r_pantilt_adapter/meshes/v1_combined/center.dae"  />
 				</geometry>
-			</collision>
+			</collision>-->
 			<inertial>
 				<mass value="0.025" />
@@ -56,5 +56,5 @@
 	<joint name="pantilt_tilt_joint" type="revolute">
       <axis xyz="1 0 0"/>
-      <limit lower="0" upper="1" effort="9" velocity="1" />
+      <limit lower="0" upper="3.14" effort="9" velocity="1" />
       <origin xyz="0.0223 0 0.0455" rpy="0 0 0" />
       <parent link="pantilt_center_link"/>
@@ -67,9 +67,10 @@
 				</geometry>
 			</visual>
-			<collision name="pantilt_top_link_collision">
+	<!--		<collision name="pantilt_top_link_collision">
 				<geometry>
 					<mesh filename="package://h4r_pantilt_adapter/meshes/v1_combined/multicamera_mount.dae"  />
 				</geometry>
 			</collision>
+-->
 			<inertial>
 				<mass value="0.010" />
@@ -87,5 +88,5 @@
 		<commandTopic>cmd_dir</commandTopic>
 		<servoTorque>1.0</servoTorque>
-		<servoRate>5.0</servoRate>
+		<servoRate>500.0</servoRate>
 		<panStart>90</panStart>
 		<tiltStart>90</tiltStart>

Commit message: update xacro file to new locations of meshes

File: h4r_pantilt_descriptions/defs/pan_tilt_adapter.xacro (robot description, xacro)
@@ -3,15 +3,15 @@
        xmlns:interface="http://playerstage.sourceforge.net/gazebo/xmlschema/#interface"
        xmlns:xacro="http://ros.org/wiki/xacro"
-	   name="pan_tilt_adapter"
+	   name="pan_tilt_base_v1"
 	>
 		 <link name="pantilt_base_link">
 			<visual>
 				<geometry>
-			  		<mesh filename="package://h4r_pantilt_adapter/meshes/v1_combined/base.dae"  />
+			  		<mesh filename="package://h4r_pantilt_descriptions/mesh/dae/base_v1.dae"  />
 				</geometry>
 			</visual>
 			<collision name="pantilt_foot_link_collision">
 				<geometry>
-					<mesh filename="package://h4r_pantilt_adapter/meshes/v1_combined/base.dae"  />
+					<mesh filename="package://h4r_pantilt_descriptions/mesh/dae/base_v1.dae"  />
 				</geometry>
 			</collision>
@@ -36,10 +36,10 @@
 			<visual>
 				<geometry>
-			  		<mesh filename="package://h4r_pantilt_adapter/meshes/v1_combined/center.dae"  />
+			  		<mesh filename="package://h4r_pantilt_descriptions/mesh/dae/center_v1.dae"  />
 				</geometry>
 			</visual>
 <!--			<collision name="pantilt_center_link_collision">
 				<geometry>
-					<mesh filename="package://h4r_pantilt_adapter/meshes/v1_combined/center.dae"  />
+					<mesh filename="package://h4r_pantilt_descriptions/mesh/dae/center_v1.dae"  />
 				</geometry>
 			</collision>-->
@@ -64,10 +64,10 @@
 			<visual>
 				<geometry>
-			  		<mesh filename="package://h4r_pantilt_adapter/meshes/v1_combined/multicamera_mount.dae"  />
+			  		<mesh filename="package://h4r_pantilt_descriptions/mesh/dae/thermapp_camera_mount_v1.dae"  />
 				</geometry>
 			</visual>
 	<!--		<collision name="pantilt_top_link_collision">
 				<geometry>
-					<mesh filename="package://h4r_pantilt_adapter/meshes/v1_combined/multicamera_mount.dae"  />
+					<mesh filename="package://h4r_pantilt_descriptions/mesh/dae/thermapp_camera_mount_v1.dae"  />
 				</geometry>
 			</collision>
