Commit message: move code into separate files

File: h4r_pantilt_descriptions/defs/center/center_v1.xacro (robot description, xacro)
@@ -3,15 +3,14 @@
        xmlns:interface="http://playerstage.sourceforge.net/gazebo/xmlschema/#interface"
        xmlns:xacro="http://ros.org/wiki/xacro"
-	   name="pantilt_base_v1"
+	   name="pantilt_center_v1"
 	>
-		 <link name="pantilt_base_link">
+	<link name="pantilt_center_link">
 			<visual>
-				<origin rpy="0 0 0" xyz="0 0 0"/>
 				<geometry>
-			  		<mesh filename="package://h4r_pantilt_descriptions/mesh/dae/base_v1.dae"  />
+			  		<mesh filename="package://h4r_pantilt_descriptions/mesh/dae/center_v1.dae"  />
 				</geometry>
 			</visual>
-			<collision name="pantilt_foot_link_collision">
-				<origin rpy="0 0 0" xyz="0 0 0.0009"/>
+			<collision name="pantilt_center_link_collision">
+				<origin rpy="0 0 0" xyz="0 0 0.0026"/>
 				<geometry>
 					<cylinder length="0.0018" radius="0.045"/>
@@ -19,12 +18,12 @@
 			</collision>
 			<inertial>
-				<mass value="0.010" />
-				<inertia ixx="3.8"
-						 iyy="3.8"
-						 izz="7.6"
+				<mass value="0.025" />
+				<inertia ixx="9.325"
+						 iyy="11.911"
+						 izz="7.028"
 				         iyz="0.0"
 				         ixy="0.0"
-				         ixz="0.0" />
+				         ixz="1.025" />
 			</inertial>
-		</link>
+	</link>
 </robot>

File: h4r_pantilt_descriptions/defs/v1_thermapp_camera.xacro (robot description, xacro)
@@ -13,26 +13,5 @@
       <child link="pantilt_center_link"/>
     </joint>
-	<link name="pantilt_center_link">
-			<visual>
-				<geometry>
-			  		<mesh filename="package://h4r_pantilt_descriptions/mesh/dae/center_v1.dae"  />
-				</geometry>
-			</visual>
-			<collision name="pantilt_center_link_collision">
-				<origin rpy="0 0 0" xyz="0 0 0.0026"/>
-				<geometry>
-					<cylinder length="0.0018" radius="0.045"/>
-				</geometry>
-			</collision>
-			<inertial>
-				<mass value="0.025" />
-				<inertia ixx="9.325"
-						 iyy="11.911"
-						 izz="7.028"
-				         iyz="0.0"
-				         ixy="0.0"
-				         ixz="1.025" />
-			</inertial>
-		</link>
+    <xacro:include filename="$(find h4r_pantilt_descriptions)/defs/center/center_v1.xacro"/>
 	<joint name="pantilt_tilt_joint" type="revolute">
       <axis xyz="1 0 0"/>
@@ -40,29 +19,7 @@
       <origin xyz="0.0223 0 0.0455" rpy="0 0 0" />
       <parent link="pantilt_center_link"/>
-      <child link="pantilt_top_link"/>
+      <child link="pantilt_head_link"/>
     </joint>
-		<link name="pantilt_top_link">
-			<visual>
-				<geometry>
-			  		<mesh filename="package://h4r_pantilt_descriptions/mesh/dae/thermapp_camera_mount_v1.dae"  />
-				</geometry>
-			</visual>
-<!--
-			<collision name="pantilt_top_link_collision">
-				<geometry>
-					<mesh filename="package://h4r_pantilt_descriptions/mesh/dae/thermapp_camera_mount_v1.dae"  />
-				</geometry>
-			</collision>
--->
-			<inertial>
-				<mass value="0.010" />
-				<inertia ixx="4.481"
-						 iyy="2.930"
-						 izz="5.819"
-				         iyz="-0.083"
-				         ixy="0.049"
-				         ixz="0.317" />
-			</inertial>
-		</link>
+    <xacro:include filename="$(find h4r_pantilt_descriptions)/defs/head/head_thermapp_v1.xacro"/>
 <gazebo>
 	<plugin name="H4RPanTiltGazebo"

Commit message: fix collisions for center part v1

File: h4r_pantilt_descriptions/defs/center/center_v1.xacro (robot description, xacro)
@@ -14,5 +14,5 @@
 				<origin rpy="0 0 0" xyz="0 0 0.0026"/>
 				<geometry>
-					<cylinder length="0.0018" radius="0.045"/>
+					<cylinder length="0.0018" radius="0.040"/>
 				</geometry>
 			</collision>
@@ -27,3 +27,15 @@
 			</inertial>
 	</link>
+    <joint name="pantilt_center_col2_joint" type="fixed">
+	  <origin rpy="0 0 0" xyz="-0.00340 0 0.02955"/>
+      <parent link="pantilt_center_link"/>
+      <child link="pantilt_center_col_link"/>
+    </joint>
+	<link name="pantilt_center_col_link">
+		<collision name="pantilt_center_link_collision2">
+			<geometry>
+				<box size="0.054 0.016 0.052" />
+			</geometry>
+		</collision>
+	</link>
 </robot>
