Commit message: add posibility to have multiple adapters by adding camera name (untested)

File: h4r_pantilt_descriptions/defs/base/base_v1.xacro (robot description, xacro)
@@ -5,5 +5,5 @@
 	   name="pantilt_base_v1"
 	>
-		 <link name="pantilt_base_link">
+		 <link name="${camera_name}/pantilt_base_link">
 			<visual>
 				<origin rpy="0 0 0" xyz="0 0 0"/>
@@ -12,5 +12,5 @@
 				</geometry>
 			</visual>
-			<collision name="pantilt_foot_link_collision">
+			<collision name="${camera_name}/pantilt_base_link_collision">
 				<origin rpy="0 0 0" xyz="0 0 0.0009"/>
 				<geometry>

File: h4r_pantilt_descriptions/defs/center/center_v1.xacro (robot description, xacro)
@@ -5,5 +5,5 @@
 	   name="pantilt_center_v1"
 	>
-	<link name="pantilt_center_link">
+	<link name="${camera_name}/pantilt_center_link">
 			<visual>
 				<geometry>
@@ -11,5 +11,5 @@
 				</geometry>
 			</visual>
-			<collision name="pantilt_center_link_collision">
+			<collision name="${camera_name}/pantilt_center_link_collision">
 				<origin rpy="0 0 0" xyz="0 0 0.0026"/>
 				<geometry>
@@ -27,11 +27,11 @@
 			</inertial>
 	</link>
-    <joint name="pantilt_center_col2_joint" type="fixed">
+    <joint name="${camera_name}/pantilt_center_col2_joint" type="fixed">
 	  <origin rpy="0 0 0" xyz="-0.00340 0 0.02955"/>
-      <parent link="pantilt_center_link"/>
-      <child link="pantilt_center_col_link"/>
+      <parent link="${camera_name}/pantilt_center_link"/>
+      <child link="${camera_name}/pantilt_center_col_link"/>
     </joint>
-	<link name="pantilt_center_col_link">
-		<collision name="pantilt_center_link_collision2">
+	<link name="${camera_name}/pantilt_center_col_link">
+		<collision name="${camera_name}/pantilt_center_link_collision2">
 			<geometry>
 				<box size="0.054 0.016 0.052" />

File: h4r_pantilt_descriptions/defs/head/head_thermapp_v1.xacro (robot description, xacro)
@@ -5,5 +5,5 @@
 	   name="head_thermapp_v1"
 	>
-		<link name="pantilt_head_link">
+		<link name="${camera_name}/pantilt_head_link">
 			<visual>
 				<geometry>
@@ -11,5 +11,5 @@
 				</geometry>
 			</visual>
-			<collision name="pantilt_top_link_collision">
+			<collision name="${camera_name}/pantilt_head_link_collision">
 			    <origin rpy="0 -1.57079632679 0" xyz="-0.0168 0.00606 -0.00335"/>
 				<geometry>

File: h4r_pantilt_descriptions/defs/v1_thermapp_camera.xacro (robot description, xacro)
@@ -5,23 +5,25 @@
 	   name="pan_tilt_thermapp_camera"
 	>
+	<xacro:arg name="camera_name" default="cam"/>
+	<property name="camera_name" value="$(arg camera_name)" />
 	<xacro:include filename="$(find h4r_pantilt_descriptions)/defs/base/base_v1.xacro"/>
-	<joint name="pantilt_pan_joint" type="revolute">
+	<joint name="${camera_name}/pantilt_pan_joint" type="revolute">
       <axis xyz="0 0 1"/>
       <limit lower="0" upper="3.14" effort="9" velocity="1" />
       <origin xyz="0 0 0.0027" rpy="0 0 0" />
-      <parent link="pantilt_base_link"/>
-      <child link="pantilt_center_link"/>
+      <parent link="${camera_name}/pantilt_base_link"/>
+      <child link="${camera_name}/pantilt_center_link"/>
     </joint>
     <xacro:include filename="$(find h4r_pantilt_descriptions)/defs/center/center_v1.xacro"/>
-	<joint name="pantilt_tilt_joint" type="revolute">
+	<joint name="${camera_name}/pantilt_tilt_joint" type="revolute">
       <axis xyz="1 0 0"/>
       <limit lower="0" upper="3.14" effort="9" velocity="1" />
       <origin xyz="0.0223 0 0.0455" rpy="0 0 0" />
-      <parent link="pantilt_center_link"/>
-      <child link="pantilt_head_link"/>
+      <parent link="${camera_name}/pantilt_center_link"/>
+      <child link="${camera_name}/pantilt_head_link"/>
     </joint>
     <xacro:include filename="$(find h4r_pantilt_descriptions)/defs/head/head_thermapp_v1.xacro"/>
 <gazebo>
-	<plugin name="H4RPanTiltGazebo"
+	<plugin name="${camera_name}/H4RPanTiltGazebo"
 		filename="libh4r_pantilt_gazebo.so">
 		<commandTopic>cmd_dir</commandTopic>
@@ -30,6 +32,6 @@
 		<panStart>90</panStart>
 		<tiltStart>90</tiltStart>
-		<panJoint>pantilt_pan_joint</panJoint>
-		<tiltJoint>pantilt_tilt_joint</tiltJoint>
+		<panJoint>${camera_name}/pantilt_pan_joint</panJoint>
+		<tiltJoint>${camera_name}/pantilt_tilt_joint</tiltJoint>
 		<alwaysOn>true</alwaysOn>
 	</plugin>
