Commit message: add collision to thermapp head

File: h4r_pantilt_descriptions/defs/head/head_thermapp_v1.xacro (robot description, xacro)
@@ -12,6 +12,7 @@
 			</visual>
 			<collision name="pantilt_top_link_collision">
+			    <origin rpy="0 -1.57079632679 0" xyz="-0.0168 0.00606 -0.00335"/>
 				<geometry>
-					<mesh filename="package://h4r_pantilt_descriptions/mesh/dae/thermapp_camera_mount_v1.dae"  />
+					<box size="0.061 0.037 0.039" />
 				</geometry>
 			</collision>

Commit message: add h4r_rapid_robot xacros add macro for PI

File: h4r_pantilt_descriptions/defs/head/head_thermapp_v1.xacro (robot description, xacro)
@@ -12,5 +12,5 @@
 			</visual>
 			<collision name="${camera_name}/pantilt_head_link_collision">
-			    <origin rpy="0 -1.57079632679 0" xyz="-0.0168 0.00606 -0.00335"/>
+			    <origin rpy="0 -${rr_const_pi/2} 0" xyz="-0.0168 0.00606 -0.00335"/>
 				<geometry>
 					<box size="0.061 0.037 0.039" />

File: h4r_pantilt_descriptions/defs/v1_thermapp_camera.xacro (robot description, xacro)
@@ -7,8 +7,9 @@
 	<xacro:arg name="camera_name" default="cam"/>
 	<property name="camera_name" value="$(arg camera_name)" />
+	<xacro:include filename="$(find h4r_rapid_robot_xacros)/defs/rapid_robot.xacro"/>
 	<xacro:include filename="$(find h4r_pantilt_descriptions)/defs/base/base_v1.xacro"/>
 	<joint name="${camera_name}/pantilt_pan_joint" type="revolute">
       <axis xyz="0 0 1"/>
-      <limit lower="0" upper="3.14" effort="9" velocity="1" />
+      <limit lower="0" upper="${rr_const_pi}" effort="9" velocity="1" />
       <origin xyz="0 0 0.0027" rpy="0 0 0" />
       <parent link="${camera_name}/pantilt_base_link"/>
@@ -18,5 +19,5 @@
 	<joint name="${camera_name}/pantilt_tilt_joint" type="revolute">
       <axis xyz="1 0 0"/>
-      <limit lower="0" upper="3.14" effort="9" velocity="1" />
+      <limit lower="0" upper="${rr_const_pi}" effort="9" velocity="1" />
       <origin xyz="0.0223 0 0.0455" rpy="0 0 0" />
       <parent link="${camera_name}/pantilt_center_link"/>
