Commit message: add camera plugin

File: h4r_pantilt_descriptions/defs/head/head_delock_96000_v1.xacro (robot description, xacro)
@@ -3,27 +3,39 @@
        xmlns:interface="http://playerstage.sourceforge.net/gazebo/xmlschema/#interface"
        xmlns:xacro="http://ros.org/wiki/xacro"
-	   name="head_thermapp_v1"
+	   name="head_delock_96000_v1"
 	>
-		<link name="${camera_name}/pantilt_head_link">
-			<visual>
-				<geometry>
-			  		<mesh filename="package://h4r_pantilt_descriptions/mesh/dae/delock_96000_camera_mount_v1.dae"  />
-				</geometry>
-			</visual>
-			<collision name="${camera_name}/pantilt_head_link_collision">
-			    <origin rpy="${rr_const_pi/2} 0 ${rr_const_pi/2*3}" xyz="-0.0203 0.0084 0.0"/>
-				<geometry>
-					<box size="0.027 0.01 0.06" />
-				</geometry>
-			</collision>
-			<inertial>
-				<mass value="0.010" />
-				<inertia ixx="4.481"
-						 iyy="2.930"
-						 izz="5.819"
-				         iyz="-0.083"
-				         ixy="0.049"
-				         ixz="0.317" />
-			</inertial>
-		</link>
+	<xacro:include filename="$(find h4r_hardware_models)/defs/models.xacro"/>
+	<!-- camera model -->
+	<xacro:hw_models_delock_96000
+			 camera_name="${camera_name}"
+			 frame_id="${camera_name}"
+	 />
+	<joint name="${camera_name}/pantilt_head_camera_joint" type="fixed">
+	  <origin rpy="-${rr_const_pi/2} 0 -${rr_const_pi}" xyz="-0.0223 0.0218 0"/>
+      <parent link="${camera_name}/pantilt_head_link"/>
+      <child link="${camera_name}/mesh"/>
+    </joint>
+	<!--pantilt head-->
+	<link name="${camera_name}/pantilt_head_link">
+		<visual>
+			<geometry>
+		  		<mesh filename="package://h4r_pantilt_descriptions/mesh/dae/delock_96000_camera_mount_v1.dae"  />
+			</geometry>
+		</visual>
+		<collision name="${camera_name}/pantilt_head_link_collision">
+		    <origin rpy="${rr_const_pi/2} 0 ${rr_const_pi/2*3}" xyz="-0.0203 0.0084 0.0"/>
+			<geometry>
+				<box size="0.027 0.01 0.06" />
+			</geometry>
+		</collision>
+		<inertial>
+			<mass value="0.010" />
+			<inertia ixx="4.481"
+					 iyy="2.930"
+					 izz="5.819"
+			         iyz="-0.083"
+			         ixy="0.049"
+			         ixz="0.317" />
+		</inertial>
+	</link>
 </robot>

Commit message: add macro for v1 delock 96000 add pantilt robot add robot launch file

File: h4r_pantilt_descriptions/defs/head/head_delock_96000_v1.xacro (robot description, xacro)
@@ -5,5 +5,4 @@
 	   name="head_delock_96000_v1"
 	>
-	<xacro:include filename="$(find h4r_hardware_models)/defs/models.xacro"/>
 	<!-- camera model -->
 	<xacro:hw_models_delock_96000

File: h4r_pantilt_descriptions/defs/v1_delock_96000.xacro (robot description, xacro)
@@ -7,22 +7,8 @@
 	<xacro:arg name="camera_name" default="cam"/>
 	<property name="camera_name" value="$(arg camera_name)" />
+	<xacro:include filename="$(find h4r_hardware_models)/defs/models.xacro"/>
 	<xacro:include filename="$(find h4r_rapid_robot_xacros)/defs/rapid_robot.xacro"/>
-	<xacro:include filename="$(find h4r_pantilt_descriptions)/defs/base/base_v1.xacro"/>
-	<joint name="${camera_name}/pantilt_pan_joint" type="revolute">
-      <axis xyz="0 0 1"/>
-      <limit lower="0" upper="${rr_const_pi}" effort="9" velocity="1" />
-      <origin xyz="0 0 0.0027" rpy="0 0 0" />
-      <parent link="${camera_name}/pantilt_base_link"/>
-      <child link="${camera_name}/pantilt_center_link"/>
-    </joint>
-    <xacro:include filename="$(find h4r_pantilt_descriptions)/defs/center/center_v1.xacro"/>
-	<joint name="${camera_name}/pantilt_tilt_joint" type="revolute">
-      <axis xyz="1 0 0"/>
-      <limit lower="0" upper="${rr_const_pi}" effort="9" velocity="1" />
-      <origin xyz="0.0223 0 0.0455" rpy="0 0 0" />
-      <parent link="${camera_name}/pantilt_center_link"/>
-      <child link="${camera_name}/pantilt_head_link"/>
-    </joint>
-    <xacro:include filename="$(find h4r_pantilt_descriptions)/defs/head/head_delock_96000_v1.xacro"/>
-	<xacro:include filename="$(find h4r_pantilt_descriptions)/defs/gazebo/v1_gazebo.xacro"/>
+	<xacro:include filename="$(find h4r_pantilt_descriptions)/defs/robot_macro/m_v1_delock96000.xacro"/>
+	<xacro:h4r_pantilt_v1
+		camera_name="$(arg camera_name)" />
 </robot>
