Commit message: reformat descriptions

File: h4r_pantilt_descriptions/def/base/base_v1.xacro (robot description, xacro)
@@ -3,28 +3,27 @@
        xmlns:interface="http://playerstage.sourceforge.net/gazebo/xmlschema/#interface"
        xmlns:xacro="http://ros.org/wiki/xacro"
-	   name="pantilt_base_v1"
-	>
-		 <link name="${camera_name}/pantilt_base_link">
-			<visual>
-				<origin rpy="0 0 0" xyz="0 0 0"/>
-				<geometry>
-			  		<mesh filename="package://h4r_pantilt_descriptions/mesh/dae/base_v1.dae"  />
-				</geometry>
-			</visual>
-			<collision name="${camera_name}/pantilt_base_link_collision">
-				<origin rpy="0 0 0" xyz="0 0 0.0009"/>
-				<geometry>
-					<cylinder length="0.0018" radius="0.045"/>
-				</geometry>
-			</collision>
-			<inertial>
-				<mass value="0.010" />
-				<inertia ixx="3.8"
-						 iyy="3.8"
-						 izz="7.6"
-				         iyz="0.0"
-				         ixy="0.0"
-				         ixz="0.0" />
-			</inertial>
-		</link>
+	   name="pantilt_base_v1">
+ <link name="${camera_name}/pantilt_base_link">
+	<visual>
+		<origin rpy="0 0 0" xyz="0 0 0"/>
+		<geometry>
+	  		<mesh filename="package://h4r_pantilt_descriptions/mesh/dae/base_v1.dae"  />
+		</geometry>
+	</visual>
+	<collision name="${camera_name}/pantilt_base_link_collision">
+		<origin rpy="0 0 0" xyz="0 0 0.0009"/>
+		<geometry>
+			<cylinder length="0.0018" radius="0.045"/>
+		</geometry>
+	</collision>
+	<inertial>
+		<mass value="0.010" />
+		<inertia ixx="3.8"
+				 iyy="3.8"
+				 izz="7.6"
+		         iyz="0.0"
+		         ixy="0.0"
+		         ixz="0.0" />
+	</inertial>
+</link>
 </robot>

File: h4r_pantilt_descriptions/def/center/center_v1.xacro (robot description, xacro)
@@ -5,37 +5,37 @@
 	   name="pantilt_center_v1"
 	>
-	<link name="${camera_name}/pantilt_center_link">
-			<visual>
-				<geometry>
-			  		<mesh filename="package://h4r_pantilt_descriptions/mesh/dae/center_v1.dae"  />
-				</geometry>
-			</visual>
-			<collision name="${camera_name}/pantilt_center_link_collision">
-				<origin rpy="0 0 0" xyz="0 0 0.0026"/>
-				<geometry>
-					<cylinder length="0.0018" radius="0.040"/>
-				</geometry>
-			</collision>
-			<inertial>
-				<mass value="0.025" />
-				<inertia ixx="9.325"
-						 iyy="11.911"
-						 izz="7.028"
-				         iyz="0.0"
-				         ixy="0.0"
-				         ixz="1.025" />
-			</inertial>
-	</link>
-    <joint name="${camera_name}/pantilt_center_col2_joint" type="fixed">
-	  <origin rpy="0 0 0" xyz="-0.00340 0 0.02955"/>
-      <parent link="${camera_name}/pantilt_center_link"/>
-      <child link="${camera_name}/pantilt_center_col_link"/>
-    </joint>
-	<link name="${camera_name}/pantilt_center_col_link">
-		<collision name="${camera_name}/pantilt_center_link_collision2">
-			<geometry>
-				<box size="0.054 0.016 0.052" />
-			</geometry>
-		</collision>
-	</link>
+<link name="${camera_name}/pantilt_center_link">
+	<visual>
+		<geometry>
+	  		<mesh filename="package://h4r_pantilt_descriptions/mesh/dae/center_v1.dae"  />
+		</geometry>
+	</visual>
+	<collision name="${camera_name}/pantilt_center_link_collision">
+		<origin rpy="0 0 0" xyz="0 0 0.0026"/>
+		<geometry>
+			<cylinder length="0.0018" radius="0.040"/>
+		</geometry>
+	</collision>
+	<inertial>
+		<mass value="0.025" />
+		<inertia ixx="9.325"
+				 iyy="11.911"
+				 izz="7.028"
+		         iyz="0.0"
+		         ixy="0.0"
+		         ixz="1.025" />
+	</inertial>
+</link>
+<joint name="${camera_name}/pantilt_center_col2_joint" type="fixed">
+  <origin rpy="0 0 0" xyz="-0.00340 0 0.02955"/>
+  <parent link="${camera_name}/pantilt_center_link"/>
+  <child link="${camera_name}/pantilt_center_col_link"/>
+</joint>
+<link name="${camera_name}/pantilt_center_col_link">
+	<collision name="${camera_name}/pantilt_center_link_collision2">
+		<geometry>
+			<box size="0.054 0.016 0.052" />
+		</geometry>
+	</collision>
+</link>
 </robot>

File: h4r_pantilt_descriptions/def/gazebo/v1_gazebo.xacro (robot description, xacro)
@@ -10,5 +10,5 @@
 		<commandTopic>${camera_name}/cmd_dir</commandTopic>
 		<servoTorque>1.0</servoTorque>
-		<servoRate>500.0</servoRate>
+		<servoRate>125</servoRate>
 		<panStart>90</panStart>
 		<tiltStart>90</tiltStart>

File: h4r_pantilt_descriptions/def/head/head_delock_96000_v1.xacro (robot description, xacro)
@@ -5,36 +5,36 @@
 	   name="head_delock_96000_v1"
 	>
-	<!-- camera model -->
-	<xacro:hw_models_delock_96000
-			 camera_name="${camera_name}"
-			 frame_id="${camera_name}"
-	 />
-	<joint name="${camera_name}/pantilt_head_camera_joint" type="fixed">
-	  <origin rpy="-${rr_const_pi/2} 0 -${rr_const_pi}" xyz="-0.0223 0.0218 0"/>
-      <parent link="${camera_name}/pantilt_head_link"/>
-      <child link="${camera_name}/mesh"/>
-    </joint>
-	<!--pantilt head-->
-	<link name="${camera_name}/pantilt_head_link">
-		<visual>
-			<geometry>
-		  		<mesh filename="package://h4r_pantilt_descriptions/mesh/dae/delock_96000_camera_mount_v1.dae"  />
-			</geometry>
-		</visual>
-		<collision name="${camera_name}/pantilt_head_link_collision">
-		    <origin rpy="${rr_const_pi/2} 0 ${rr_const_pi/2*3}" xyz="-0.0203 0.0084 0.0"/>
-			<geometry>
-				<box size="0.027 0.01 0.06" />
-			</geometry>
-		</collision>
-		<inertial>
-			<mass value="0.010" />
-			<inertia ixx="4.481"
-					 iyy="2.930"
-					 izz="5.819"
-			         iyz="-0.083"
-			         ixy="0.049"
-			         ixz="0.317" />
-		</inertial>
-	</link>
+<!-- camera model -->
+<xacro:hw_models_delock_96000
+		 camera_name="${camera_name}"
+		 frame_id="${camera_name}"
+ />
+<joint name="${camera_name}/pantilt_head_camera_joint" type="fixed">
+  <origin rpy="-${rr_const_pi/2} 0 -${rr_const_pi}" xyz="-0.0223 0.0218 0"/>
+  <parent link="${camera_name}/pantilt_head_link"/>
+  <child link="${camera_name}/mesh"/>
+</joint>
+<!--pantilt head-->
+<link name="${camera_name}/pantilt_head_link">
+	<visual>
+		<geometry>
+	  		<mesh filename="package://h4r_pantilt_descriptions/mesh/dae/delock_96000_camera_mount_v1.dae"  />
+		</geometry>
+	</visual>
+	<collision name="${camera_name}/pantilt_head_link_collision">
+	    <origin rpy="${rr_const_pi/2} 0 ${rr_const_pi/2*3}" xyz="-0.0203 0.0084 0.0"/>
+		<geometry>
+			<box size="0.027 0.01 0.06" />
+		</geometry>
+	</collision>
+	<inertial>
+		<mass value="0.010" />
+		<inertia ixx="4.481"
+				 iyy="2.930"
+				 izz="5.819"
+		         iyz="-0.083"
+		         ixy="0.049"
+		         ixz="0.317" />
+	</inertial>
+</link>
 </robot>

File: h4r_pantilt_descriptions/def/robot_macro/m_v1_delock96000.xacro (robot description, xacro)
@@ -10,5 +10,5 @@
 	<joint name="${camera_name}/pantilt_pan_joint" type="revolute">
       <axis xyz="0 0 1"/>
-      <limit lower="0" upper="${rr_const_pi}" effort="9" velocity="1" />
+      <limit lower="0" upper="${rr_const_pi}" effort="0.1" velocity="1" />
       <origin xyz="0 0 0.0027" rpy="0 0 0" />
       <parent link="${camera_name}/pantilt_base_link"/>
@@ -18,5 +18,5 @@
 	<joint name="${camera_name}/pantilt_tilt_joint" type="revolute">
       <axis xyz="1 0 0"/>
-      <limit lower="0" upper="${rr_const_pi}" effort="9" velocity="1" />
+      <limit lower="0" upper="${rr_const_pi}" effort="0.1" velocity="1" />
       <origin xyz="0.0223 0 0.0455" rpy="0 0 0" />
       <parent link="${camera_name}/pantilt_center_link"/>
